File: board/steelseries-rival310.sch (KiCad schematic (older format))
At the start: 11 parts, among them SW1 BTN_LEFT, SW2 BTN_RIGHT, SW3 BTN_DPI, SW3 BTN_WHEEL, SW4 BTN_BACK, SW5 BTN_FORWARD, U1 STM32F103T6Ux, U2 TUREMOVE3

Commit message: schematic cleanup
Parts:
- D1: renamed from D2; symbol steelseries-rival310-rescue:LED_RGB-Device -> steelseries-rival310-rescue:LED_RGB-Device-steelseries-rival310-rescue
- D2: renamed from D1; symbol steelseries-rival310-rescue:LED_RGB-Device -> steelseries-rival310-rescue:LED_RGB-Device-steelseries-rival310-rescue
- ENC1: renamed from SW?; symbol steelseries-rival310-rescue:Rotary_Encoder-Device -> steelseries-rival310-rescue:Rotary_Encoder-Device-steelseries-rival310-rescue
- SW1, SW2, SW3: symbol steelseries-rival310-rescue:SW_Push_Open-Switch -> steelseries-rival310-rescue:SW_Push_Open-Switch-steelseries-rival310-rescue
- SW4: renamed from SW3; symbol steelseries-rival310-rescue:SW_Push_Open-Switch -> steelseries-rival310-rescue:SW_Push_Open-Switch-steelseries-rival310-rescue
- SW5: renamed from SW4; symbol steelseries-rival310-rescue:SW_Push_Open-Switch -> steelseries-rival310-rescue:SW_Push_Open-Switch-steelseries-rival310-rescue
- SW6: renamed from SW5; symbol steelseries-rival310-rescue:SW_Push_Open-Switch -> steelseries-rival310-rescue:SW_Push_Open-Switch-steelseries-rival310-rescue
- U1: symbol steelseries-rival310-rescue:STM32F103T6Ux-MCU_ST_STM32F1 -> steelseries-rival310-rescue:STM32F103T6Ux-MCU_ST_STM32F1-steelseries-rival310-rescue
- U2: symbol steelseries-rival310-rescue:TUREMOVE3-steelseries -> steelseries-rival310-rescue:TUREMOVE3-steelseries-steelseries-rival310-rescue
Connections:
- net labels added: BTN_BACK, BTN_DPI, BTN_FORWARD, BTN_LEFT, BTN_RIGHT, BTN_WHEEL, ENC_A, ENC_B, LED_LOGO_BLUE, LED_LOGO_GREEN, LED_LOGO_RED, LED_WHEEL_BLUE, LED_WHEEL_GREEN, LED_WHEEL_RED, SPI_CLK, SPI_CS, SPI_MISO, SPI_MOSI, TRUEMOVE3_MOTION
- net labels removed: FLASH_CS
Other:
- note added: "Flash"
- note added: "Inverted"
- moved on the sheet: D1, D2, ENC1, SW1, SW2, SW3, SW4, SW5, SW6

Commit message: update README, added rival dump of external eeprom
Other:
- note added: "External EEPROM"
- note added: "Through transistors"
- note removed: "Flash"
- moved on the sheet: D1, D2, ENC1, SW1, SW2, SW3, SW4, SW5, SW6, U2
